File: qse2.kicad_pcb (KiCad board)
At the start: 2 copper layers, 100 x 75 mm, 71 parts, among them J1 5-1814832-1, J2 5-1814832-1, J3 Conn_02x08_Odd_Even, J4 SJ-3524-SMT, J6 Conn_01x02, U1 SN74LVC1G14DBV, U2 SN74LVC1G14DBV, U3 SN74CBT3253, U4 SN74AC74PW, U5 AD8137ARZ-R7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

Commit message: Added description of Audio Adapter changes to README.md.
Other:
- board text removed: "3.3V"
Changed lines of the file:
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@@
-		)
-	)
-	(gr_text "3.3V"
-		(at 129.125 82.675 0)
-		(layer "F.SilkS")
-		(effects
-			(font
-				(size 1 1)
-				(thickness 0.15)
-			)
-			(justify left bottom)
 		)
 	)
@@
 	)
 	(gr_text "5.0V"
-		(at 129.4 76.15 0)
+		(at 123.5 79.2 0)
 		(layer "F.SilkS")
 		(effects
