File: qse2.kicad_pcb (KiCad board)
At the start: 2 copper layers, 100 x 75 mm, 81 parts, among them J1 5-1814832-1, J2 5-1814832-1, J3 Conn_02x08_Odd_Even, J4 SJ-3524-SMT, J6 Conn_01x02, J7 B4B-XH-A_LF__SN_, U1 SN74LVC1G14DBV, U10 SN74LVC1G14DBV, U11 NCP508SQ33T1G, U2 SN74LVC1G14DBV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

Commit message: Swapped SDA and SCL to correct pins.
Parts:
- U11: value NCP508SQ33T1G -> NCP114ASN330T1G
- U6: value NCP115ASN330T2G -> NCV8114ASN165T1G
Connections:
- J7 pad 3: /SCL -> /SDA
- J7 pad 4: /SDA -> /SCL
Routing:
- net /SDA: track 137.5 -> 138.6 mm
- net /SCL: track 138.1 -> 137.2 mm, vias 0 -> 1
Other:
- board text added: "V1.2"
- board text removed: "V1.1"
