File: qse2.kicad_pcb (KiCad board)
At the start: 2 copper layers, 100 x 75 mm, 81 parts, among them J1 5-1814832-1, J2 5-1814832-1, J3 Conn_02x08_Odd_Even, J4 SJ-3524-SMT, J6 Conn_01x02, J7 B4B-XH-A_LF__SN_, U1 SN74LVC1G14DBV, U10 SN74LVC1G14DBV, U11 NCP114ASN330T1G, U2 SN74LVC1G14DBV, U3 SN74CBT3253, U4 SN74AC74PW, U5 AD8137ARZ-R7, U6 NCV8114ASN165T1G, U7 UA78M05IDCYR, U8 AP2120N-2.5TRG1, U9 AD8137ARZ-R7

Commit message: Ready for release to fab.
Parts:
- removed C2: 0.1uF, Capacitor_SMD:C_1206_3216Metric
- removed C26: 1uF, Capacitor_SMD:C_1206_3216Metric
- removed R3: DNP, Resistor_SMD:R_1206_3216Metric
- removed R9: 1k, Resistor_SMD:R_1206_3216Metric
- added C18: 0.01uF, Capacitor_SMD:C_1206_3216Metric, F.Cu at (111.1, 88.3)
- added C30: 1uF, Capacitor_SMD:C_1206_3216Metric, F.Cu at (147.6, 92.8)
- added C32: 1uF, Capacitor_SMD:C_1206_3216Metric, F.Cu at (152.8, 81.2)
- added R37: 2.2k, Resistor_SMD:R_1206_3216Metric, F.Cu at (156.3, 88.8)
- added TP3: TestPoint, Connector_PinHeader_2.54mm:PinHeader_1x01_P2.54mm_Vertical, F.Cu at (194.4, 67.4)
- C27: value 1uF -> 10uF
- C8: value 0.1uF -> 0.01uF
- U6: value NCV8114ASN165T1G -> AP7343; footprint 16TSOP:TSOP-5-483-N_ONS -> Package_TO_SOT_SMD:TSOT-23-5
- U8: value AP2120N-2.5TRG1 -> REF3016E; footprint AP2120N:SOT-23_DIO -> Package_TO_SOT_SMD:SOT-23-3
- moved U6 7.94 mm to (156.9, 84.9)
- moved U8 6.31 mm to (152.4, 91.6)
Connections:
- U5 pad 7: /TXRX_OA -> unconnected-(U5-PD_NOT-Pad7)
- U6 pad 5: /REF1.6 -> /REF_I
- U8 pad 1: GND -> /5V_FILT
- U8 pad 2: /REF_I -> /REF1.6
- U8 pad 3: /5V_FILT -> GND
- U9 pad 7: /TXRX_OA -> unconnected-(U9-PD_NOT-Pad7)
Routing:
- net /TXRX_OA: track 61.7 -> 0.00 mm, vias 4 -> 0
- net /TXRX: track 64.1 -> 40.9 mm
- net GND: track 21.0 -> 33.6 mm, vias 150 -> 146
- net /REF_I: track 38.6 -> 41.4 mm
- net /5V_FILT: track 206.9 -> 204.3 mm, vias 7 -> 8
- net /REF1.6: track 68.9 -> 66.4 mm
- net /SDA: track 138.6 -> 140.1 mm
Other:
- board text added: "5V"
- board text added: "GND"
- board text added: "SCL"
- board text added: "SDA"
