File: qse2.kicad_pcb (KiCad board)
At the start: 2 copper layers, 100 x 75 mm, 81 parts, among them J1 5-1814832-1, J2 5-1814832-1, J3 Conn_02x08_Odd_Even, J4 SJ-3524-SMT, J6 Conn_01x02, J7 B4B-XH-A_LF__SN_, U1 SN74LVC1G14DBV, U10 SN74LVC1G14DBV, U11 NCP508SQ33T1G, U2 SN74LVC1G14DBV, U3 SN74CBT3253, U4 SN74AC74PW, U5 AD8137ARZ-R7, U6 NCP115ASN330T2G, U7 UA78M05IDCYR, U8 AP2120N-2.5TRG1, U9 AD8137ARZ-R7

Commit message: Fixed flip-flop part number.
Parts:
- U11: value NCP508SQ33T1G -> NCP114ASN330T1G
- U4: value SN74AC74PW -> SN74LVC74ADR
- U6: value NCP115ASN330T2G -> NCV8114ASN165T1G
